File: pcb/switch.kicad_sch (KiCad schematic)
At the start: 10 parts, among them Q2 AO3400A, Q3 AO3400A, Q4 AO3400A, SW4 SW_Push

Commit message: Layout except stm32
Parts:
- removed R10: 150, Resistor_SMD:R_0603_1608Metric, symbol Device:R
- added R7: 150, Resistor_SMD:R_0603_1608Metric, symbol Device:R
- renumbered D2 to D1, D3 to D2, D4 to D3, Q2 to Q1, Q3 to Q2, Q4 to Q3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
Connections:
- net VBUS: now also R7.1
- net at D1.2 (A): now also R7.2
