File: pcb/switch-panel.kicad_pcb (KiCad board)
At the start: 2 copper layers, 73.3 x 35.4 mm, 58 parts, among them J1 USB_C_Receptacle_USB2.0_16P, J2 Conn_ARM_SWD_TagConnect_TC203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, Q1 AO3400A, Q2 AO3400A, Q3 AO3400A, Q4 AO3400A, Q5 AO3400A, Q6 AO3400A, Q7 AO3400A, Q8 AO3400A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

Commit message: Add test production files
Parts:
- moved C4 29.7 mm to (76.5, 90.7), turned to -90 degrees
- moved C5 12.8 mm to (86.3, 87.9)
- moved Y1 11.9 mm to (90.9, 92.1)
- moved C12 11.7 mm to (93.6, 92.1), turned to -90 degrees
- moved C6 10.4 mm to (89.3, 96.0), turned to 90 degrees
- moved C11 9.04 mm to (90.9, 89.8)
- moved R4 8.86 mm to (90.9, 94.4)
- moved U3 7.98 mm to (82.8, 94.0)
- moved C3 5.29 mm to (76.6, 98.7), turned to -90 degrees
- moved R3 4.18 mm to (84.3, 87.9), turned to 0 degrees
- moved C10 2.52 mm to (90.9, 96.0), turned to 0 degrees
- moved C7 2.09 mm to (78.4, 99.2), turned to -90 degrees

Commit message: Final routing and production
Parts:
- moved J2 13.3 mm to (121.8, 95.2), turned to 90 degrees
- moved C4 0.26 mm to (76.6, 90.4)
- turned C10 to 180 degrees
Connections:
- U3 pad 13: /BTN1 -> unconnected-(U3-PA3-Pad13)
- U3 pad 19: unconnected-(U3-PB1-Pad19) -> /BTN1
Routing:
- net +3V3: track 17.5 -> 113.2 mm, vias 0 -> 1
- net /LEDB3: track 0.00 -> 62.7 mm, vias 0 -> 2
- net /SWDIO: track 0.00 -> 62.3 mm, vias 0 -> 2
- net /BTN2: track 0.00 -> 55.4 mm, vias 0 -> 1
- net /SWCLK: track 0.00 -> 54.2 mm
- net /LEDG3: track 0.00 -> 52.4 mm, vias 0 -> 2
- net /SWO: track 0.00 -> 48.4 mm
- net /LEDR3: track 0.00 -> 46.6 mm, vias 0 -> 2
- net /BTN3: track 0.00 -> 44.4 mm, vias 0 -> 1
- net /RST: track 0.00 -> 42.2 mm, vias 0 -> 2
- net VBUS: track 116.6 -> 76.0 mm
- net /LEDG2: track 0.00 -> 40.6 mm, vias 0 -> 2
- net /LEDB1: track 0.00 -> 40.2 mm, vias 0 -> 2
- net /SCL: track 2.03 -> 40.9 mm
- net /SDA: track 2.03 -> 40.7 mm
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