File: pcb/switch-panel.kicad_sch (KiCad schematic)
At the start: 34 parts, among them J1 Conn_ARM_SWD_TagConnect_TC203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, J2 USB_C_Receptacle_USB2.0_16P, SW1 SW_Push, SW2 SW_Push, SW3 SW_Push, U1 STM32F103C8Tx, U2 SRV05-4, U3 AMS1117-3.3, U4 SSD1306, Y1 16MHz

Commit message: Setup stm32 cube
Parts:
- removed SW1, SW2, SW3: SW_Push, symbol Switch:SW_Push
- R5, R6: footprint (none) -> Resistor_SMD:R_0402_1005Metric
Connections:
- net BTN1: now also U1.13 (PA3); no longer U1.10 (PA0)
- net BTN2: now also U1.14 (PA4); no longer U1.11 (PA1)
- net BTN3: now also U1.15 (PA5); no longer U1.12 (PA2)
- net LEDR3: now reaches U1.16 (PA6)
- net LEDG3: now reaches U1.17 (PA7)
- net LEDB3: now reaches U1.18 (PB0)
- net LEDR1: now reaches U1.29 (PA8)
- net LEDG1: now reaches U1.30 (PA9)
- net LEDB1: now reaches U1.31 (PA10)
- new net LEDB2: U1.12 (PA2)
- new net LEDG2: U1.11 (PA1)
- new net LEDR2: U1.10 (PA0)
- no-connect marks 29 -> 20
Other:
- added sheet Switch1 (switch.kicad_sch)
- added sheet Switch2 (switch.kicad_sch)
- added sheet Switch3 (switch.kicad_sch)

Commit message: Layout except stm32
Parts:
- removed C12: 22u, Capacitor_SMD:C_0603_1608Metric, symbol Device:C
- removed H4: MountingHole, MountingHole:MountingHole_3.2mm_M3, symbol Mechanical:MountingHole
- removed L1: 2u2, Inductor_SMD:L_0805_2012Metric, symbol Device:L
- renumbered C10 to C1, C1 to C10, C2 to C11, C3 to C12, C9 to C13, C11 to C2, C4 to C3, C5 to C4, C6 to C5, C7 to C6, C8 to C7, C13 to C9, J2 to J1, J1 to J2, R6 to R1, R5 to R2, R1 to R3, R2 to R4, R3 to R5, R4 to R6, U3 to U1, U4 to U2, U1 to U3, U2 to U4
Connections:
- net OPWR is gone; now on net +3V3: C9.1, U2.3 (VCC)

Commit message: Final routing and production
Connections:
- net BTN1: now also U3.19 (PB1); no longer U3.13 (PA3)
- no-connect marks 20 -> 19
Changed lines of the file:
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@@
-	)
-	(no_connect
-		(at 86.36 119.38)
 	)
 	(no_connect
@@
 	(wire
 		(pts
+			(xy 80.01 119.38) (xy 86.36 119.38)
+		)
+		(stroke
+			(width 0)
+			(type default)
+		)
+	)
+	(wire
+		(pts
 			(xy 106.68 81.28) (xy 106.68 83.82)
 		)
@@
 		(pts
 			(xy 38.1 73.66) (xy 38.1 76.2)
-		)
-		(stroke
-			(width 0)
-			(type default)
-		)
-	)
-	(wire
-		(pts
-			(xy 119.38 96.52) (xy 124.46 96.52)
 		)
 		(stroke
@@
 		)
 	)
+	(label "BTN1"
+		(at 80.01 119.38 0)
+		(fields_autoplaced yes)
+		(effects
+			(font
+				(size 1.27 1.27)
+			)
+			(justify left bottom)
+		)
+	)
 	(label "LEDR3"
 		(at 120.65 104.14 0)
@@
 		(fields_autoplaced yes)
 		(effects
-			(font
-				(size 1.27 1.27)
-			)
-			(justify left bottom)
-		)
-	)
-	(label "BTN1"
-		(at 120.65 96.52 0)
-		(fields_autoplaced yes)
-		(effects
